File: evnotipi.kicad_pcb (KiCad board)
At the start: 2 copper layers, 35.6 x 39.4 mm, 23 parts, among them J1 Conn_01x04, J2 Conn_01x03, U1 LM393, U2 LM393

Commit message: Fine adjust voltage splitter
Parts:
- R1, R3: value R27K -> R22K
Changed lines of the file:
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@@
       (effects (font (size 1 1) (thickness 0.15)))
     )
-    (fp_text value R27K (at 3.81 2.37 180) (layer F.Fab)
+    (fp_text value R22K (at 3.81 2.37 180) (layer F.Fab)
       (effects (font (size 1 1) (thickness 0.15)))
     )
@@
       (effects (font (size 1 1) (thickness 0.15)))
     )
-    (fp_text value R27K (at 3.81 2.37 180) (layer F.Fab)
+    (fp_text value R22K (at 3.81 2.37 180) (layer F.Fab)
       (effects (font (size 1 1) (thickness 0.15)))
     )
